Commit message: preparing for submission

File: src/my_robot/urdf/my_robot.xacro (robot description, xacro)
@@ -7,5 +7,8 @@
   <xacro:property name="base_width" value="0.3"/>
   <xacro:property name="base_length" value="0.4"/>
-  <xacro:property name="wheel_body_space" value="0.14"/>
+  <xacro:property name="wheel_body_space" value="0.18"/>
+  <xacro:property name="top_heigth" value="0.05"/>
+  <xacro:property name="top_width" value="0.2"/>
+  <xacro:property name="top_length" value="0.3"/>
   <link name="robot_footprint"></link>
   <xacro:include filename="$(find my_robot)/urdf/my_robot.gazebo" />
@@ -39,4 +42,33 @@
     </visual>
   </link>
+   <link name='chassis_top'>
+    <inertial>
+      <mass value="5.0"/>
+      <origin xyz="0.0 0 0" rpy=" 0 0 0"/>
+      <inertia
+          ixx="0.1" ixy="0" ixz="0"
+          iyy="0.1" iyz="0"
+          izz="0.1"
+      />
+    </inertial>
+    <collision name='chassis_top_collision'>
+      <origin xyz="0 0 0" rpy=" 0 0 0"/>
+      <geometry>
+        <box size="${top_length} ${top_width} ${top_heigth}"/>
+      </geometry>
+    </collision>
+    <visual name='chassis_top_visual'>
+      <origin xyz="0 0 0" rpy=" 0 0 0"/>
+      <geometry>
+        <box size="${top_length} ${top_width} ${top_heigth}"/>
+      </geometry>
+    </visual>
+  </link>
+  <joint type="fixed" name="chassis_top_joint">
+		<origin xyz="0 0 0.05" rpy="0 0 0"/>
+		<child link="chassis_top"/>
+		<parent link="chassis"/>
+		<axis xyz="0 1 0" rpy="0 0 0"/>
+  </joint>
   <link name="left_rear_wheel">
   	<inertial>
@@ -222,7 +254,7 @@
 	</link>
 	<joint type="fixed" name="hokuyo-joint">
-		<origin xyz="0.15 0 0.1" rpy="0 0 0"/>
+		<origin xyz="0.1 0 0.05" rpy="0 0 0"/>
 		<child link="hokuyo"/>
-		<parent link="chassis"/>
+		<parent link="chassis_top"/>
 		<axis xyz="0 1 0" rpy="0 0 0"/>
 	</joint>
@@ -242,3 +274,6 @@
 		<material>Gazebo/Blue</material>
 	</gazebo>
+	<gazebo reference="chassis_top">
+		<material>Gazebo/Red</material>
+	</gazebo>
 </robot>

Commit message: config updates

File: src/my_robot/urdf/my_robot.xacro (robot description, xacro)
@@ -219,9 +219,9 @@
 	</link>
 	<joint name="camera_optical_joint" type="fixed">
-            <origin xyz="0 0 0" rpy="-1.5708 0 -1.5708"/>
+            <origin xyz="0 0 0" rpy="-1.5707 0 -1.5707"/>
             <parent link="camera"/>
-            <child link="camera_frame_optical"/>
+            <child link="camera_link_optical"/>
         </joint>
-        <link name="camera_frame_optical"/>
+        <link name="camera_link_optical"/>
 	<joint type="fixed" name="camera-joint">
 		<origin xyz="0.25 0 0.05" rpy="0 0 0"/>
